File: msp430-nrf24.sch (EAGLE design)
At the start: 12 parts, among them IC1 MSP430G2X53-20N20, IC2 78L33, J1 PWR

Commit message: Fixed routing and dc barrel jack
Parts:
- J1: device SparkFun-Connectors:POWER_JACKSLT -> SparkFun-Connectors:POWER_JACKPTH
Changed lines of the file:
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@@
 <part name="IC2" library="SparkFun-PowerIC" deviceset="V_REG_78XX" device="TO-92_UNTESTED" value="78L33"/>
 <part name="C2" library="SparkFun-Passives" deviceset="CAP_POL" device="PTH2" value="10uF"/>
-<part name="J1" library="SparkFun-Connectors" deviceset="POWER_JACK" device="SLT" value="PWR"/>
+<part name="J1" library="SparkFun-Connectors" deviceset="POWER_JACK" device="PTH" value="PWR"/>
 <part name="GND2" library="SparkFun-Aesthetics" deviceset="GND" device=""/>
 <part name="SUPPLY2" library="SparkFun-Aesthetics" deviceset="VCC" device=""/>

Commit message: :new: Change board layout
Parts:
- removed JP1: H1, SparkFun-Connectors:M06LOCK
- removed JP2: H2, SparkFun-Connectors:M05LOCK
- removed JP3: nRF24L01, SparkFun-Connectors:M04X2
- removed JP4: H3, SparkFun-Connectors:M03LOCK
- added SV1: (no value), con-lstb:MA03-1
- added SV2: (no value), con-lstb:MA05-1
- added SV3: (no value), con-lstb:MA06-1
- added SV4: (no value), con-lstb:MA04-2
Connections:
- net CE: now also SV4.5; no longer JP3.4
- net CSN: now also SV4.6; no longer JP3.3
- net GND: now also SV2.5, SV4.7; no longer JP2.5, JP3.2
- net IRQ: now also SV4.2; no longer JP3.7
- net MISO: now also SV4.1; no longer JP3.8
- net MOSI: now also SV4.4; no longer JP3.5
- net P1.0: now also SV3.5; no longer JP1.5
- net P1.1: now also SV3.4; no longer JP1.4
- net P1.2: now also SV3.3; no longer JP1.3
- net P1.3: now also SV3.2; no longer JP1.2
- net P1.4: now also SV3.1; no longer JP1.1
- net P2.3: now also SV1.1; no longer JP4.1
- net P2.4: now also SV1.2; no longer JP4.2
- net P2.5: now also SV1.3; no longer JP4.3
- net P2.6: now also SV2.4; no longer JP2.4
- net P2.7: now also SV2.3; no longer JP2.3
- net RST: now also SV2.1; no longer JP2.1
- net SCK: now also SV4.3; no longer JP3.6
- net TEST: now also SV2.2; no longer JP2.2
- net VCC: now also SV3.6, SV4.8; no longer JP1.6, JP3.1
Changed lines of the file:
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@@
 <?xml version="1.0" encoding="utf-8"?>
 <!DOCTYPE eagle SYSTEM "eagle.dtd">
-<eagle version="7.1.0">
+<eagle version="7.2.0">
 <drawing>
 <settings>
@@
 <attributes>
 <attribute name="CNAME" value="MSP430G2553 With nRF24L01 Header"/>
-<attribute name="CREVISION" value="0.1"/>
+<attribute name="CREVISION" value="0.2"/>
 <attribute name="DESIGNER" value="RNDC"/>
 </attributes>
@@
 <part name="R1" library="SparkFun-Passives" deviceset="RESISTOR" device="KIT" value="47K"/>
 <part name="S1" library="SparkFun-Electromechanical" deviceset="TAC_SWITCH" device="PTH" value="Reset"/>
-<part name="JP3" library="SparkFun-Connectors" deviceset="M04X2" device="" value="nRF24L01"/>
 <part name="SUPPLY1" library="SparkFun-Aesthetics" deviceset="VCC" device=""/>
 <part name="GND1" library="SparkFun-Aesthetics" deviceset="GND" device=""/>
-<part name="JP1" library="SparkFun-Connectors" deviceset="M06" device="LOCK" value="H1"/>
-<part name="JP2" library="SparkFun-Connectors" deviceset="M05" device="LOCK" value="H2"/>
-<part name="JP4" library="SparkFun-Connectors" deviceset="M03" device="LOCK" value="H3"/>
 <part name="IC2" library="SparkFun-PowerIC" deviceset="V_REG_78XX" device="TO-92_UNTESTED" value="78L33"/>
 <part name="C2" library="SparkFun-Passives" deviceset="CAP_POL" device="PTH2" value="10uF"/>
@@
 <part name="SUPPLY2" library="SparkFun-Aesthetics" deviceset="VCC" device=""/>
 <part name="C3" library="SparkFun-Passives" deviceset="CAP_POL" device="PTH2" value="1uF"/>
+<part name="SV1" library="con-lstb" deviceset="MA03-1" device=""/>
+<part name="SV2" library="con-lstb" deviceset="MA05-1" device=""/>
+<part name="SV3" library="con-lstb" deviceset="MA06-1" device=""/>
+<part name="SV4" library="con-lstb" deviceset="MA04-2" device=""/>
 </parts>
 <sheets>
@@
 <instance part="R1" gate="G$1" x="7.62" y="2.54" rot="R180"/>
 <instance part="S1" gate="S" x="43.18" y="30.48" rot="R90"/>
-<instance part="JP3" gate="G$1" x="10.16" y="-12.7"/>
 <instance part="SUPPLY1" gate="G$1" x="-25.4" y="50.8"/>
 <instance part="GND1" gate="1" x="50.8" y="-17.78"/>
-<instance part="JP1" gate="G$1" x="-43.18" y="27.94"/>
-<instance part="JP2" gate="G$1" x="71.12" y="30.48" rot="MR0"/>
-<instance part="JP4" gate="G$1" x="71.12" y="10.16" rot="MR0"/>
 <instance part="IC2" gate="G$1" x="68.58" y="68.58"/>
 <instance part="C2" gate="G$1" x="55.88" y="63.5"/>
@@
 <instance part="SUPPLY2" gate="G$1" x="81.28" y="71.12"/>
 <instance part="C3" gate="G$1" x="81.28" y="63.5"/>
+<instance part="SV1" gate="G$1" x="71.12" y="10.16" rot="MR0"/>
+<instance part="SV2" gate="G$1" x="71.12" y="30.48" rot="MR0"/>
+<instance part="SV3" gate="1" x="-45.72" y="30.48"/>
+<instance part="SV4" gate="G$1" x="10.16" y="-10.16"/>
 </instances>
 <busses>
@@
 </segment>
 <segment>
-<pinref part="JP2" gate="G$1" pin="1"/>
 <wire x1="63.5" y1="25.4" x2="60.96" y2="25.4" width="0.1524" layer="91"/>
 <label x="60.96" y="25.4" size="1.27" layer="95" rot="MR0" xref="yes"/>
+<pinref part="SV2" gate="G$1" pin="1"/>
 </segment>
 </net>
 <net name="CSN" class="0">
 <segment>
-<pinref part="JP3" gate="G$1" pin="3"/>
 <wire x1="2.54" y1="-10.16" x2="0" y2="-10.16" width="0.1524" layer="91"/>
 <label x="0" y="-10.16" size="1.27" layer="95" rot="MR0" xref="yes"/>
+<pinref part="SV4" gate="G$1" pin="6"/>
 </segment>
 <segment>
@@
 <net name="MOSI" class="0">
 <segment>
-<pinref part="JP3" gate="G$1" pin="5"/>
 <wire x1="2.54" y1="-12.7" x2="0" y2="-12.7" width="0.1524" layer="91"/>
 <label x="0" y="-12.7" size="1.27" layer="95" rot="MR0" xref="yes"/>
+<pinref part="SV4" gate="G$1" pin="4"/>
 </segment>
 <segment>
@@
 <net name="IRQ" class="0">
 <segment>
-<pinref part="JP3" gate="G$1" pin="7"/>
 <wire x1="2.54" y1="-15.24" x2="0" y2="-15.24" width="0.1524" layer="91"/>
 <label x="0" y="-15.24" size="1.27" layer="95" rot="MR0" xref="yes"/>
+<pinref part="SV4" gate="G$1" pin="2"/>
 </segment>
 <segment>
@@
 <net name="CE" class="0">
 <segment>
-<pinref part="JP3" gate="G$1" pin="4"/>
 <wire x1="17.78" y1="-10.16" x2="20.32" y2="-10.16" width="0.1524" layer="91"/>
 <label x="20.32" y="-10.16" size="1.27" layer="95" xref="yes"/>
+<pinref part="SV4" gate="G$1" pin="5"/>
 </segment>
 <segment>
@@
 <net name="SCK" class="0">
 <segment>
-<pinref part="JP3" gate="G$1" pin="6"/>
 <wire x1="17.78" y1="-12.7" x2="20.32" y2="-12.7" width="0.1524" layer="91"/>
 <label x="20.32" y="-12.7" size="1.27" layer="95" xref="yes"/>
+<pinref part="SV4" gate="G$1" pin="3"/>
 </segment>
 <segment>
@@
 <net name="MISO" class="0">
 <segment>
-<pinref part="JP3" gate="G$1" pin="8"/>
 <wire x1="17.78" y1="-15.24" x2="20.32" y2="-15.24" width="0.1524" layer="91"/>
 <label x="20.32" y="-15.24" size="1.27" layer="95" xref="yes"/>
+<pinref part="SV4" gate="G$1" pin="1"/>
 </segment>
 <segment>
@@
 <wire x1="-22.86" y1="35.56" x2="-25.4" y2="35.56" width="0.1524" layer="91"/>
 <wire x1="-25.4" y1="35.56" x2="-25.4" y2="50.8" width="0.1524" layer="91"/>
-<pinref part="JP3" gate="G$1" pin="1"/>
 <wire x1="2.54" y1="-7.62" x2="-25.4" y2="-7.62" width="0.1524" layer="91"/>
 <wire x1="-25.4" y1="-7.62" x2="-25.4" y2="35.56" width="0.1524" layer="91"/>
 <junction x="-25.4" y="35.56"/>
-</segment>
-<segment>
-<pinref part="JP1" gate="G$1" pin="6"/>
+<pinref part="SV4" gate="G$1" pin="8"/>
+</segment>
+<segment>
 <wire x1="-38.1" y1="35.56" x2="-35.56" y2="35.56" width="0.1524" layer="91"/>
 <label x="-35.56" y="35.56" size="1.27" layer="95" xref="yes"/>
+<pinref part="SV3" gate="1" pin="6"/>
 </segment>
 <segment>
@@
 <wire x1="45.72" y1="35.56" x2="50.8" y2="35.56" width="0.1524" layer="91"/>
 <wire x1="50.8" y1="35.56" x2="50.8" y2="-7.62" width="0.1524" layer="91"/>
-<pinref part="JP3" gate="G$1" pin="2"/>
 <wire x1="50.8" y1="-7.62" x2="50.8" y2="-15.24" width="0.1524" layer="91"/>
 <wire x1="17.78" y1="-7.62" x2="50.8" y2="-7.62" width="0.1524" layer="91"/>
@@
 <pinref part="S1" gate="S" pin="4"/>
 <junction x="45.72" y="35.56"/>
-</segment>
-<segment>
-<pinref part="JP2" gate="G$1" pin="5"/>
+<pinref part="SV4" gate="G$1" pin="7"/>
+</segment>
+<segment>
 <wire x1="63.5" y1="35.56" x2="60.96" y2="35.56" width="0.1524" layer="91"/>
 <label x="60.96" y="35.56" size="1.27" layer="95" rot="MR0" xref="yes"/>
+<pinref part="SV2" gate="G$1" pin="5"/>
 </segment>
 <segment>
@@
 </segment>
 <segment>
-<pinref part="JP1" gate="G$1" pin="5"/>
 <wire x1="-38.1" y1="33.02" x2="-35.56" y2="33.02" width="0.1524" layer="91"/>
 <label x="-35.56" y="33.02" size="1.27" layer="95" xref="yes"/>
+<pinref part="SV3" gate="1" pin="5"/>
 </segment>
 </net>
@@
 </segment>
 <segment>
-<pinref part="JP1" gate="G$1" pin="4"/>
 <wire x1="-38.1" y1="30.48" x2="-35.56" y2="30.48" width="0.1524" layer="91"/>
 <label x="-35.56" y="30.48" size="1.27" layer="95" xref="yes"/>
+<pinref part="SV3" gate="1" pin="4"/>
 </segment>
 </net>
@@
 </segment>
 <segment>
-<pinref part="JP1" gate="G$1" pin="3"/>
 <wire x1="-38.1" y1="27.94" x2="-35.56" y2="27.94" width="0.1524" layer="91"/>
 <label x="-35.56" y="27.94" size="1.27" layer="95" xref="yes"/>
+<pinref part="SV3" gate="1" pin="3"/>
 </segment>
 </net>
@@
 </segment>
 <segment>
-<pinref part="JP1" gate="G$1" pin="2"/>
 <wire x1="-38.1" y1="25.4" x2="-35.56" y2="25.4" width="0.1524" layer="91"/>
 <label x="-35.56" y="25.4" size="1.27" layer="95" xref="yes"/>
+<pinref part="SV3" gate="1" pin="2"/>
 </segment>
 </net>
@@
 </segment>
 <segment>
-<pinref part="JP1" gate="G$1" pin="1"/>
 <wire x1="-38.1" y1="22.86" x2="-35.56" y2="22.86" width="0.1524" layer="91"/>
 <label x="-35.56" y="22.86" size="1.27" layer="95" xref="yes"/>
+<pinref part="SV3" gate="1" pin="1"/>
 </segment>
 </net>
@@
 </segment>
 <segment>
-<pinref part="JP4" gate="G$1" pin="3"/>
 <wire x1="63.5" y1="12.7" x2="60.96" y2="12.7" width="0.1524" layer="91"/>
 <label x="60.96" y="12.7" size="1.27" layer="95" rot="MR0" xref="yes"/>
+<pinref part="SV1" gate="G$1" pin="3"/>
 </segment>
 </net>
@@
 </segment>
 <segment>
-<pinref part="JP4" gate="G$1" pin="2"/>
 <wire x1="63.5" y1="10.16" x2="60.96" y2="10.16" width="0.1524" layer="91"/>
 <label x="60.96" y="10.16" size="1.27" layer="95" rot="MR0" xref="yes"/>
+<pinref part="SV1" gate="G$1" pin="2"/>
 </segment>
 </net>
@@
 </segment>
 <segment>
-<pinref part="JP4" gate="G$1" pin="1"/>
 <wire x1="63.5" y1="7.62" x2="60.96" y2="7.62" width="0.1524" layer="91"/>
 <label x="60.96" y="7.62" size="1.27" layer="95" rot="MR0" xref="yes"/>
+<pinref part="SV1" gate="G$1" pin="1"/>
 </segment>
 </net>
@@
 </segment>
 <segment>
-<pinref part="JP2" gate="G$1" pin="2"/>
 <wire x1="63.5" y1="27.94" x2="60.96" y2="27.94" width="0.1524" layer="91"/>
 <label x="60.96" y="27.94" size="1.27" layer="95" rot="MR0" xref="yes"/>
+<pinref part="SV2" gate="G$1" pin="2"/>
 </segment>
 </net>
@@
 </segment>
 <segment>
-<pinref part="JP2" gate="G$1" pin="3"/>
 <wire x1="63.5" y1="30.48" x2="60.96" y2="30.48" width="0.1524" layer="91"/>
 <label x="60.96" y="30.48" size="1.27" layer="95" rot="MR0" xref="yes"/>
+<pinref part="SV2" gate="G$1" pin="3"/>
 </segment>
 </net>
@@
 </segment>
 <segment>
-<pinref part="JP2" gate="G$1" pin="4"/>
 <wire x1="63.5" y1="33.02" x2="60.96" y2="33.02" width="0.1524" layer="91"/>
 <label x="60.96" y="33.02" size="1.27" layer="95" rot="MR0" xref="yes"/>
-</segment>
-</net>
+<pinref part="SV2" gate="G$1" pin="4"/>
+</segment>
+</net>
